Commit message: update

File: src/RelaxedIK/urdfs/kinova_two_arm.urdf (robot description, URDF)
Before this commit: robot dual_robot, 21 links, 20 joints
Joints:
- joint fixed_camera: origin xyz=0 0 0 rpy=0 -1.57 0 -> xyz=0 0 0 rpy=0 -1.57 3.14

Commit message: update

File: src/RelaxedIK/urdfs/kinova_two_arm.urdf (robot description, URDF)
Before this commit: robot dual_robot, 21 links, 20 joints
Links:
- link leftbase_link: geometry collision mesh filename=package://relaxed_ik/kortex_description/arms/gen3/7dof/mesh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; visual mesh filename=package://relaxed_ik/kortex_description/arms/gen3/7dof/mesh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
- link leftbracelet_link: geometry collision mesh filename=package://relaxed_ik/kortex_description/arms/gen3/7dof/mesh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; visual mesh filename=package://relaxed_ik/kortex_description/arms/gen3/7dof/mesh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
- link leftforearm_link: geometry collision mesh filename=package://relaxed_ik/kortex_description/arms/gen3/7dof/mesh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; visual mesh filename=package://relaxed_ik/kortex_description/arms/gen3/7dof/mesh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
- link lefthalf_arm_1_link: geometry collision mesh filename=package://relaxed_ik/kortex_description/arms/gen3/7dof/mesh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; visual mesh filename=package://relaxed_ik/kortex_description/arms/gen3/7dof/mesh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
- link lefthalf_arm_2_link: geometry collision mesh filename=package://relaxed_ik/kortex_description/arms/gen3/7dof/mesh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; visual mesh filename=package://relaxed_ik/kortex_description/arms/gen3/7dof/mesh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
- link leftshoulder_link: geometry collision mesh filename=package://relaxed_ik/kortex_description/arms/gen3/7dof/mesh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; visual mesh filename=package://relaxed_ik/kortex_description/arms/gen3/7dof/mesh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
- link leftspherical_wrist_1_link: geometry collision mesh filename=package://relaxed_ik/kortex_description/arms/gen3/7dof/mesh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; visual mesh filename=package://relaxed_ik/kortex_description/arms/gen3/7dof/mesh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
- link leftspherical_wrist_2_link: geometry collision mesh filename=package://relaxed_ik/kortex_description/arms/gen3/7dof/mesh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; visual mesh filename=package://relaxed_ik/kortex_description/arms/gen3/7dof/mesh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
- link rightbase_link: geometry collision mesh filename=package://relaxed_ik/kortex_description/arms/gen3/7dof/mesh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; visual mesh filename=package://relaxed_ik/kortex_description/arms/gen3/7dof/mesh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
- link rightbracelet_link: geometry collision mesh filename=package://relaxed_ik/kortex_description/arms/gen3/7dof/mesh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; visual mesh filename=package://relaxed_ik/kortex_description/arms/gen3/7dof/mesh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
- link rightforearm_link: geometry collision mesh filename=package://relaxed_ik/kortex_description/arms/gen3/7dof/mesh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; visual mesh filename=package://relaxed_ik/kortex_description/arms/gen3/7dof/mesh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
- link righthalf_arm_1_link: geometry collision mesh filename=package://relaxed_ik/kortex_description/arms/gen3/7dof/mesh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; visual mesh filename=package://relaxed_ik/kortex_description/arms/gen3/7dof/mesh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
- link righthalf_arm_2_link: geometry collision mesh filename=package://relaxed_ik/kortex_description/arms/gen3/7dof/mesh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; visual mesh filename=package://relaxed_ik/kortex_description/arms/gen3/7dof/mesh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
- link rightshoulder_link: geometry collision mesh filename=package://relaxed_ik/kortex_description/arms/gen3/7dof/mesh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; visual mesh filename=package://relaxed_ik/kortex_description/arms/gen3/7dof/mesh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
- link rightspherical_wrist_1_link: geometry collision mesh filename=package://relaxed_ik/kortex_description/arms/gen3/7dof/mesh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; visual mesh filename=package://relaxed_ik/kortex_description/arms/gen3/7dof/mesh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
- link rightspherical_wrist_2_link: geometry collision mesh filename=package://relaxed_ik/kortex_description/arms/gen3/7dof/mesh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; visual mesh filename=package://relaxed_ik/kortex_description/arms/gen3/7dof/mesh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

Commit message: update

File: src/RelaxedIK/urdfs/kinova_two_arm.urdf (robot description, URDF)
Before this commit: robot dual_robot, 21 links, 20 joints
Links:
- added link leftleft_inner_finger, mass 0.00000000104003125914103; collision mesh filename=package://relaxed_ik/kortex_description/grippers/robotiq_2f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 scale=0.001 0.001 0.001; visual mesh filename=package://relaxed_ik/kortex_description/grippers/robotiq_2f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 scale=0.001 0.001 0.001
- added link leftleft_inner_finger_pad; collision box size=0.022 0.00635 0.0375; visual box size=0.022 0.00635 0.0375
- added link leftleft_inner_knuckle, mass 0.00000000271177346495152; collision mesh filename=package://relaxed_ik/kortex_description/grippers/robotiq_2f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 scale=0.001 0.001 0.001; visual mesh filename=package://relaxed_ik/kortex_description/grippers/robotiq_2f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 scale=0.001 0.001 0.001
- added link leftleft_outer_finger, mass 0.00000000022614240507152; collision mesh filename=package://relaxed_ik/kortex_description/grippers/robotiq_2f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 scale=0.001 0.001 0.001; visual mesh filename=package://relaxed_ik/kortex_description/grippers/robotiq_2f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 scale=0.001 0.001 0.001
- added link leftleft_outer_knuckle, mass 0.00000000853198276973456; collision mesh filename=package://relaxed_ik/kortex_description/grippers/robotiq_2f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 scale=0.001 0.001 0.001; visual mesh filename=package://relaxed_ik/kortex_description/grippers/robotiq_2f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 scale=0.001 0.001 0.001
- added link leftright_inner_finger, mass 0.0000000104003125914103; collision mesh filename=package://relaxed_ik/kortex_description/grippers/robotiq_2f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 scale=0.001 0.001 0.001; visual mesh filename=package://relaxed_ik/kortex_description/grippers/robotiq_2f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 scale=0.001 0.001 0.001
- added link leftright_inner_finger_pad; collision box size=0.022 0.00635 0.0375; visual box size=0.022 0.00635 0.0375
- added link leftright_inner_knuckle, mass 0.0000000271177346495152; collision mesh filename=package://relaxed_ik/kortex_description/grippers/robotiq_2f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 scale=0.001 0.001 0.001; visual mesh filename=package://relaxed_ik/kortex_description/grippers/robotiq_2f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 scale=0.001 0.001 0.001
- added link leftright_outer_finger, mass 0.000000022614240507152; collision mesh filename=package://relaxed_ik/kortex_description/grippers/robotiq_2f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 scale=0.001 0.001 0.001; visual mesh filename=package://relaxed_ik/kortex_description/grippers/robotiq_2f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 scale=0.001 0.001 0.001
- added link leftright_outer_knuckle, mass 0.0000000853198276973456; collision mesh filename=package://relaxed_ik/kortex_description/grippers/robotiq_2f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 scale=0.001 0.001 0.001; visual mesh filename=package://relaxed_ik/kortex_description/grippers/robotiq_2f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 scale=0.001 0.001 0.001
- added link leftrobotiq_arg2f_base_link, mass 0.00022652; collision mesh filename=package://relaxed_ik/kortex_description/grippers/robotiq_2f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; visual mesh filename=package://relaxed_ik/kortex_description/grippers/robotiq_2f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
Joints:
- added joint gripper_base_joint: type fixed, parent leftend_effector_link, child leftrobotiq_arg2f_base_link, origin xyz=0.0 0.0 0.0 rpy=0.0 0.0 1.57
- added joint leftfinger_joint: type fixed, parent leftrobotiq_arg2f_base_link, child leftleft_outer_knuckle, origin xyz=0 -0.0306011 0.054904 rpy=0 0 3.14159
- added joint leftleft_inner_finger_joint: type fixed, parent leftleft_outer_finger, child leftleft_inner_finger, origin xyz=0 0.0061 0.0471 rpy=0 0 0
- added joint leftleft_inner_finger_pad_joint: type fixed, parent leftleft_inner_finger, child leftleft_inner_finger_pad, origin xyz=0 -0.0220203446692936 0.03242 rpy=0 0 0, axis 0 0 1
- added joint leftleft_inner_knuckle_joint: type fixed, parent leftrobotiq_arg2f_base_link, child leftleft_inner_knuckle, origin xyz=0 -0.0127 0.06142 rpy=0 0 3.14159
- added joint leftleft_outer_finger_joint: type fixed, parent leftleft_outer_knuckle, child leftleft_outer_finger, origin xyz=0 0.0315 -0.0041 rpy=0 0 0
- added joint leftright_inner_finger_joint: type fixed, parent leftright_outer_finger, child leftright_inner_finger, origin xyz=0 0.0061 0.0471 rpy=0 0 0
- added joint leftright_inner_finger_pad_joint: type fixed, parent leftright_inner_finger, child leftright_inner_finger_pad, origin xyz=0 -0.0220203446692936 0.03242 rpy=0 0 0
- added joint leftright_inner_knuckle_joint: type fixed, parent leftrobotiq_arg2f_base_link, child leftright_inner_knuckle, origin xyz=0 0.0127 0.06142 rpy=0 0 0
- added joint leftright_outer_finger_joint: type fixed, parent leftright_outer_knuckle, child leftright_outer_finger, origin xyz=0 0.0315 -0.0041 rpy=0 0 0
- added joint leftright_outer_knuckle_joint: type fixed, parent leftrobotiq_arg2f_base_link, child leftright_outer_knuckle, origin xyz=0 0.0306011 0.054904 rpy=0 0 0

Commit message: comitted by Ajay

File: src/RelaxedIK/urdfs/kinova_two_arm.urdf (robot description, URDF)
Before this commit: robot dual_robot, 21 links, 20 joints
Links:
- added link leftleft_inner_finger, mass 0.00000000104003125914103; collision mesh filename=package://kortex_description/grippers/robotiq_2f_85/meshes/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 scale=0.001 0.001 0.001; visual mesh filename=package://kortex_description/grippers/robotiq_2f_85/meshes/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 scale=0.001 0.001 0.001
- added link leftleft_inner_finger_pad; collision box size=0.022 0.00635 0.0375; visual box size=0.022 0.00635 0.0375
- added link leftleft_inner_knuckle, mass 0.00000000271177346495152; collision mesh filename=package://kortex_description/grippers/robotiq_2f_85/meshes/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 scale=0.001 0.001 0.001; visual mesh filename=package://kortex_description/grippers/robotiq_2f_85/meshes/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 scale=0.001 0.001 0.001
- added link leftleft_outer_finger, mass 0.00000000022614240507152; collision mesh filename=package://kortex_description/grippers/robotiq_2f_85/meshes/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 scale=0.001 0.001 0.001; visual mesh filename=package://kortex_description/grippers/robotiq_2f_85/meshes/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 scale=0.001 0.001 0.001
- added link leftleft_outer_knuckle, mass 0.00000000853198276973456; collision mesh filename=package://kortex_description/grippers/robotiq_2f_85/meshes/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 scale=0.001 0.001 0.001; visual mesh filename=package://kortex_description/grippers/robotiq_2f_85/meshes/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 scale=0.001 0.001 0.001
- added link leftright_inner_finger, mass 0.0000000104003125914103; collision mesh filename=package://kortex_description/grippers/robotiq_2f_85/meshes/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 scale=0.001 0.001 0.001; visual mesh filename=package://kortex_description/grippers/robotiq_2f_85/meshes/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 scale=0.001 0.001 0.001
- added link leftright_inner_finger_pad; collision box size=0.022 0.00635 0.0375; visual box size=0.022 0.00635 0.0375
- added link leftright_inner_knuckle, mass 0.0000000271177346495152; collision mesh filename=package://kortex_description/grippers/robotiq_2f_85/meshes/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 scale=0.001 0.001 0.001; visual mesh filename=package://kortex_description/grippers/robotiq_2f_85/meshes/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 scale=0.001 0.001 0.001
- added link leftright_outer_finger, mass 0.000000022614240507152; collision mesh filename=package://kortex_description/grippers/robotiq_2f_85/meshes/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 scale=0.001 0.001 0.001; visual mesh filename=package://kortex_description/grippers/robotiq_2f_85/meshes/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 scale=0.001 0.001 0.001
- added link leftright_outer_knuckle, mass 0.0000000853198276973456; collision mesh filename=package://kortex_description/grippers/robotiq_2f_85/meshes/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 scale=0.001 0.001 0.001; visual mesh filename=package://kortex_description/grippers/robotiq_2f_85/meshes/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 scale=0.001 0.001 0.001
- added link leftrobotiq_arg2f_base_link, mass 0.00022652; collision mesh filename=package://kortex_description/grippers/robotiq_2f_85/meshes/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; visual mesh filename=package://kortex_description/grippers/robotiq_2f_85/meshes/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
Joints:
- added joint gripper_base_joint: type fixed, parent leftend_effector_link, child leftrobotiq_arg2f_base_link, origin xyz=0.0 0.0 0.0 rpy=0.0 0.0 1.57
- added joint leftfinger_joint: type fixed, parent leftrobotiq_arg2f_base_link, child leftleft_outer_knuckle, origin xyz=0 -0.0306011 0.054904 rpy=0 0 3.14159
- added joint leftleft_inner_finger_joint: type fixed, parent leftleft_outer_finger, child leftleft_inner_finger, origin xyz=0 0.0061 0.0471 rpy=0 0 0
- added joint leftleft_inner_finger_pad_joint: type fixed, parent leftleft_inner_finger, child leftleft_inner_finger_pad, origin xyz=0 -0.0220203446692936 0.03242 rpy=0 0 0, axis 0 0 1
- added joint leftleft_inner_knuckle_joint: type fixed, parent leftrobotiq_arg2f_base_link, child leftleft_inner_knuckle, origin xyz=0 -0.0127 0.06142 rpy=0 0 3.14159
- added joint leftleft_outer_finger_joint: type fixed, parent leftleft_outer_knuckle, child leftleft_outer_finger, origin xyz=0 0.0315 -0.0041 rpy=0 0 0
- added joint leftright_inner_finger_joint: type fixed, parent leftright_outer_finger, child leftright_inner_finger, origin xyz=0 0.0061 0.0471 rpy=0 0 0
- added joint leftright_inner_finger_pad_joint: type fixed, parent leftright_inner_finger, child leftright_inner_finger_pad, origin xyz=0 -0.0220203446692936 0.03242 rpy=0 0 0
- added joint leftright_inner_knuckle_joint: type fixed, parent leftrobotiq_arg2f_base_link, child leftright_inner_knuckle, origin xyz=0 0.0127 0.06142 rpy=0 0 0
- added joint leftright_outer_finger_joint: type fixed, parent leftright_outer_knuckle, child leftright_outer_finger, origin xyz=0 0.0315 -0.0041 rpy=0 0 0
- added joint leftright_outer_knuckle_joint: type fixed, parent leftrobotiq_arg2f_base_link, child leftright_outer_knuckle, origin xyz=0 0.0306011 0.054904 rpy=0 0 0
